File: EightBitRegister/EightBitRegister.kicad_pcb (KiCad board)
At the start: 2 copper layers, 185 parts, among them J1 Conn_01x08_MountingPin, J2 Conn_01x08_MountingPin, J3 Conn_01x08_MountingPin, J4 Conn_01x08_MountingPin, J5 Conn_01x08_MountingPin, J6 Conn_01x08_MountingPin, J7 Conn_01x08_MountingPin, J8 Conn_01x08_MountingPin, J9 Conn_01x08_MountingPin, Q1 2N7000, Q10 2N7000, Q100 2N7000, Q101 2N7000, Q102 2N7000, Q103 2N7000, Q104 2N7000, Q105 2N7000, Q106 2N7000, Q107 2N7000, Q108 2N7000, Q109 2N7000, Q11 2N7000, Q110 2N7000, Q111 2N7000, Q112 2N7000, Q12 2N7000, Q13 2N7000, Q14 2N7000, Q15 2N7000, Q16 2N7000, Q17 2N7000, Q18 2N7000, Q19 2N7000, Q2 2N7000, Q20 2N7000, Q21 2N7000, Q22 2N7000, Q23 2N7000, Q24 2N7000, Q25 2N7000, Q26 2N7000, Q27 2N7000, Q28 2N7000, Q29 2N7000, Q3 2N7000, Q30 2N7000, Q31 2N7000, Q32 2N7000, Q33 2N7000, Q34 2N7000, Q35 2N7000, Q36 2N7000, Q37 2N7000, Q38 2N7000, Q39 2N7000, Q4 2N7000, Q40 2N7000, Q41 2N7000, Q42 2N7000, Q43 2N7000, Q44 2N7000, Q45 2N7000, Q46 2N7000, Q47 2N7000, Q48 2N7000, Q49 2N7000, Q5 2N7000, Q50 2N7000, Q51 2N7000, Q52 2N7000, Q53 2N7000, Q54 2N7000, Q55 2N7000, Q56 2N7000, Q57 2N7000, Q58 2N7000, Q59 2N7000, Q6 2N7000, Q60 2N7000, Q61 2N7000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

Commit message: wip
Parts:
- moved Q14 19.6 mm to (101.5, 50.4)
- moved Q5 19.6 mm to (91.5, 34.8)
- moved Q6 19.6 mm to (91.5, 40.9)
- moved Q7 19.6 mm to (91.5, 49.5)
- moved Q8 19.6 mm to (91.5, 55.6)
- moved R3 19.6 mm to (91.1, 29.2)
- moved R4 19.6 mm to (91.1, 43.9)
- moved Q10 13.1 mm to (84.5, 78.6)
- moved Q9 13.1 mm to (84.5, 72.5)
- moved R5 13.1 mm to (84.1, 67.0)
Changed lines of the file:
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@@
 	(footprint "Resistor_SMD:R_0805_2012Metric_Pad1.20x1.40mm_HandSolder"
 		(layer "F.Cu")
-		(at 71.64 31.295948 180)
+		(at 91.14 29.226224 180)
 		(descr "Resistor SMD 0805 (2012 Metric), square (rectangular) end terminal, IPC_7351 nominal with elongated pad for handsoldering. (Body size source: IPC-SM-782 page 72, https://www.pcb-3d.com/wordpress/wp-content/uploads/ipc-sm-782a_amendment_1_and_2.pdf), generated with kicad-footprint-generator")
 		(tags "resistor handsolder")
@@
 		(tags "to-92 sc-43 sc-43a sot54 PA33 transistor")
 		(property "Reference" "Q11"
-			(at 1.27 -3.56 270)
+			(at 1.27 -3.56 -90)
 			(layer "F.SilkS")
 			(effects
@@
 		)
 		(property "Value" "2N7000"
-			(at 1.27 2.79 270)
+			(at 1.27 2.79 -90)
 			(layer "F.Fab")
 			(effects
@@
 		)
 		(fp_text user "${REFERENCE}"
-			(at 1.27 0 270)
+			(at 1.27 0 -90)
 			(layer "F.Fab")
 			(effects
@@
 		(tags "to-92 sc-43 sc-43a sot54 PA33 transistor")
 		(property "Reference" "Q12"
-			(at 1.27 -3.56 270)
+			(at 1.27 -3.56 -90)
 			(layer "F.SilkS")
 			(effects
@@
 		)
 		(property "Value" "2N7000"
-			(at 1.27 2.79 270)
+			(at 1.27 2.79 -90)
 			(layer "F.Fab")
 			(effects
@@
 		)
 		(fp_text user "${REFERENCE}"
-			(at 1.27 0 270)
+			(at 1.27 0 -90)
 			(layer "F.Fab")
 			(effects
@@
 	(footprint "Resistor_SMD:R_0805_2012Metric_Pad1.20x1.40mm_HandSolder"
 		(layer "F.Cu")
-		(at 71.64 45.99378 180)
+		(at 91.14 43.924056 180)
 		(descr "Resistor SMD 0805 (2012 Metric), square (rectangular) end terminal, IPC_7351 nominal with elongated pad for handsoldering. (Body size source: IPC-SM-782 page 72, https://www.pcb-3d.com/wordpress/wp-content/uploads/ipc-sm-782a_amendment_1_and_2.pdf), generated with kicad-footprint-generator")
 		(tags "resistor handsolder")
@@
 		)
 		(property "Value" "2N7000"
-			(at 1.27 2.79 270)
+			(at 1.27 2.79 -90)
 			(layer "F.Fab")
 			(effects
@@
 		)
 		(fp_text user "${REFERENCE}"
-			(at 1.27 0 270)
+			(at 1.27 0 -90)
 			(layer "F.Fab")
 			(effects
@@
 	(footprint "Package_TO_SOT_THT:TO-92_Inline"
 		(layer "F.Cu")
-		(at 72 57.655668 90)
+		(at 91.5 55.585944 90)
 		(descr "TO-92 leads in-line, narrow, oval pads, drill 0.75mm (see NXP sot054_po.pdf)")
 		(tags "to-92 sc-43 sc-43a sot54 PA33 transistor")
 		(property "Reference" "Q8"
-			(at 1.27 -3.56 270)
+			(at 1.27 -3.56 -90)
 			(layer "F.SilkS")
 			(effects
@@
 		)
 		(property "Value" "2N7000"
-			(at 1.27 2.79 270)
+			(at 1.27 2.79 -90)
 			(layer "F.Fab")
 			(effects
@@
 		)
 		(fp_text user "${REFERENCE}"
-			(at 1.27 0 270)
+			(at 1.27 0 -90)
 			(layer "F.Fab")
 			(effects
@@
 		(tags "to-92 sc-43 sc-43a sot54 PA33 transistor")
 		(property "Reference" "Q2"
-			(at 1.27 -3.56 270)
+			(at 1.27 -3.56 -90)
 			(layer "F.SilkS")
 			(effects
@@
 		)
 		(property "Value" "2N7000"
-			(at 1.27 2.79 270)
+			(at 1.27 2.79 -90)
 			(layer "F.Fab")
 			(effects
@@
 		)
 		(fp_text user "${REFERENCE}"
-			(at 1.27 0 270)
+			(at 1.27 0 -90)
 			(layer "F.Fab")
 			(effects
@@
 	(footprint "Package_TO_SOT_THT:TO-92_Inline"
 		(layer "F.Cu")
-		(at 72 74.625948 90)
+		(at 84.5 78.625948 90)
 		(descr "TO-92 leads in-line, narrow, oval pads, drill 0.75mm (see NXP sot054_po.pdf)")
 		(tags "to-92 sc-43 sc-43a sot54 PA33 transistor")
 		(property "Reference" "Q10"
-			(at 1.27 -3.56 270)
+			(at 1.27 -3.56 -90)
 			(layer "F.SilkS")
 			(effects
@@
 		)
 		(property "Value" "2N7000"
-			(at 1.27 2.79 270)
+			(at 1.27 2.79 -90)
 			(layer "F.Fab")
 			(effects
@@
 		)
 		(fp_text user "${REFERENCE}"
-			(at 1.27 0 270)
+			(at 1.27 0 -90)
 			(layer "F.Fab")
 			(effects
@@
 	(footprint "Package_TO_SOT_THT:TO-92_Inline"
 		(layer "F.Cu")
-		(at 72 42.957836 90)
+		(at 91.5 40.888112 90)
 		(descr "TO-92 leads in-line, narrow, oval pads, drill 0.75mm (see NXP sot054_po.pdf)")
 		(tags "to-92 sc-43 sc-43a sot54 PA33 transistor")
 		(property "Reference" "Q6"
-			(at 1.27 -3.56 270)
+			(at 1.27 -3.56 -90)
 			(layer "F.SilkS")
 			(effects
@@
 		)
 		(property "Value" "2N7000"
-			(at 1.27 2.79 270)
+			(at 1.27 2.79 -90)
 			(layer "F.Fab")
 			(effects
@@
 		)
 		(fp_text user "${REFERENCE}"
-			(at 1.27 0 270)
+			(at 1.27 0 -90)
 			(layer "F.Fab")
 			(effects
@@
 	(footprint "Package_TO_SOT_THT:TO-92_Inline"
 		(layer "F.Cu")
-		(at 72 68.54 90)
+		(at 84.5 72.54 90)
 		(descr "TO-92 leads in-line, narrow, oval pads, drill 0.75mm (see NXP sot054_po.pdf)")
 		(tags "to-92 sc-43 sc-43a sot54 PA33 transistor")
 		(property "Reference" "Q9"
-			(at 1.27 -3.56 270)
+			(at 1.27 -3.56 -90)
 			(layer "F.SilkS")
 			(effects
@@
 		)
 		(property "Value" "2N7000"
-			(at 1.27 2.79 270)
+			(at 1.27 2.79 -90)
 			(layer "F.Fab")
 			(effects
@@
 		)
 		(fp_text user "${REFERENCE}"
-			(at 1.27 0 270)
+			(at 1.27 0 -90)
 			(layer "F.Fab")
 			(effects
@@
 	(footprint "Package_TO_SOT_THT:TO-92_Inline"
 		(layer "F.Cu")
-		(at 72 36.871892 90)
+		(at 91.5 34.802168 90)
 		(descr "TO-92 leads in-line, narrow, oval pads, drill 0.75mm (see NXP sot054_po.pdf)")
 		(tags "to-92 sc-43 sc-43a sot54 PA33 transistor")
 		(property "Reference" "Q5"
-			(at 1.27 -3.56 270)
+			(at 1.27 -3.56 -90)
 			(layer "F.SilkS")
 			(effects
@@
 		)
 		(property "Value" "2N7000"
-			(at 1.27 2.79 270)
+			(at 1.27 2.79 -90)
 			(layer "F.Fab")
 			(effects
@@
 		)
 		(fp_text user "${REFERENCE}"
-			(at 1.27 0 270)
+			(at 1.27 0 -90)
 			(layer "F.Fab")
 			(effects
@@
 		(tags "to-92 sc-43 sc-43a sot54 PA33 transistor")
 		(property "Reference" "Q13"
-			(at 1.27 -3.56 270)
+			(at 1.27 -3.56 -90)
 			(layer "F.SilkS")
 			(effects
@@
 		)
 		(property "Value" "2N7000"
-			(at 1.27 2.79 270)
+			(at 1.27 2.79 -90)
 			(layer "F.Fab")
 			(effects
@@
 		)
 		(fp_text user "${REFERENCE}"
-			(at 1.27 0 270)
+			(at 1.27 0 -90)
 			(layer "F.Fab")
 			(effects
@@
 	(footprint "Package_TO_SOT_THT:TO-92_Inline"
 		(layer "F.Cu")
-		(at 72 51.569724 90)
+		(at 91.5 49.5 90)
 		(descr "TO-92 leads in-line, narrow, oval pads, drill 0.75mm (see NXP sot054_po.pdf)")
 		(tags "to-92 sc-43 sc-43a sot54 PA33 transistor")
 		(property "Reference" "Q7"
-			(at 1.27 -3.56 270)
+			(at 1.27 -3.56 -90)
 			(layer "F.SilkS")
 			(effects
@@
 		)
 		(property "Value" "2N7000"
-			(at 1.27 2.79 270)
+			(at 1.27 2.79 -90)
 			(layer "F.Fab")
 			(effects
@@
 		)
 		(fp_text user "${REFERENCE}"
-			(at 1.27 0 270)
+			(at 1.27 0 -90)
 			(layer "F.Fab")
 			(effects
@@
 	(footprint "Resistor_SMD:R_0805_2012Metric_Pad1.20x1.40mm_HandSolder"
 		(layer "F.Cu")
-		(at 71.64 62.964056 180)
+		(at 84.14 66.964056 180)
 		(descr "Resistor SMD 0805 (2012 Metric), square (rectangular) end terminal, IPC_7351 nominal with elongated pad for handsoldering. (Body size source: IPC-SM-782 page 72, https://www.pcb-3d.com/wordpress/wp-content/uploads/ipc-sm-782a_amendment_1_and_2.pdf), generated with kicad-footprint-generator")
 		(tags "resistor handsolder")
@@
 		(tags "to-92 sc-43 sc-43a sot54 PA33 transistor")
 		(property "Reference" "Q1"
-			(at 1.27 -3.56 270)
+			(at 1.27 -3.56 -90)
 			(layer "F.SilkS")
 			(effects
@@
 		)
 		(property "Value" "2N7000"
-			(at 1.27 2.79 270)
+			(at 1.27 2.79 -90)
 			(layer "F.Fab")
 			(effects
@@
 		)
 		(fp_text user "${REFERENCE}"
-			(at 1.27 0 270)
+			(at 1.27 0 -90)
 			(layer "F.Fab")
 			(effects
@@
 		(tags "to-92 sc-43 sc-43a sot54 PA33 transistor")
 		(property "Reference" "Q4"
-			(at 1.27 -3.56 270)
+			(at 1.27 -3.56 -90)
 			(layer "F.SilkS")
 			(effects
@@
 		)
 		(property "Value" "2N7000"
-			(at 1.27 2.79 270)
+			(at 1.27 2.79 -90)
 			(layer "F.Fab")
 			(effects
@@
 		)
 		(fp_text user "${REFERENCE}"
-			(at 1.27 0 270)
+			(at 1.27 0 -90)
 			(layer "F.Fab")
 			(effects
@@
 	(footprint "Package_TO_SOT_THT:TO-92_Inline"
 		(layer "F.Cu")
-		(at 82 52.5)
+		(at 101.5 50.430276)
 		(descr "TO-92 leads in-line, narrow, oval pads, drill 0.75mm (see NXP sot054_po.pdf)")
 		(tags "to-92 sc-43 sc-43a sot54 PA33 transistor")
